Commit message: feat: added Camera.

File: catkin_ws/src/my_robot/urdf/my_robot.xacro (robot description, xacro)
@@ -7,4 +7,5 @@
       <child link="chassis" />
    </joint>
+   <!-- Chassis -->
    <link name="chassis">
       <pose>0 0 0.1 0 0 0</pose>
@@ -51,4 +52,5 @@
       </visual>
    </link>
+   <!-- Left Wheel -->
    <link name="left_wheel">
       <inertial>
@@ -78,4 +80,5 @@
       <dynamics damping="1.0" friction="1.0" />
    </joint>
+   <!-- Right Wheel -->
    <link name="right_wheel">
       <inertial>
@@ -105,3 +108,31 @@
       <dynamics damping="1.0" friction="1.0" />
    </joint>
+   <!-- Camera -->
+   <link name="camera">
+      <inertial>
+         <mass value="0.1" />
+         <origin xyz="0.0 0 0" rpy="0 0 0" />
+         <inertia ixx="1e-6" ixy="0" ixz="0" iyy="1e-6" iyz="0" izz="1e-6" />
+      </inertial>
+      <collision name="collision">
+         <origin xyz="0 0 0" rpy="0 0 0" />
+         <geometry>
+            <box size="0.05 0.05 0.05" />
+         </geometry>
+      </collision>
+      <visual name="camera_visual">
+         <origin xyz="0 0 0" rpy="0 0 0" />
+         <geometry>
+            <box size="0.05 0.05 0.05" />
+         </geometry>
+      </visual>
+   </link>
+   <joint type="fixed" name="camera_joint">
+      <origin xyz="0.2 0 0" rpy="0 0 0" />
+      <child link="camera" />
+      <parent link="chassis" />
+      <axis xyz="0 1 0" rpy="0 0 0" />
+      <limit effort="10000" velocity="1000" />
+      <dynamics damping="1.0" friction="1.0" />
+   </joint>
 </robot>

Commit message: feat: added Lidar and Material (Colors).

File: catkin_ws/src/my_robot/urdf/my_robot.xacro (robot description, xacro)
@@ -136,3 +136,43 @@
       <dynamics damping="1.0" friction="1.0" />
    </joint>
+   <!-- Lidar -->
+   <link name="hokuyo">
+      <inertial>
+         <mass value="1e-5" />
+         <origin xyz="0.0 0 0" rpy="0 0 0" />
+         <inertia ixx="1e-6" ixy="0" ixz="0" iyy="1e-6" iyz="0" izz="1e-6" />
+      </inertial>
+      <collision name="collision">
+         <origin xyz="0 0 0" rpy="0 0 0" />
+         <geometry>
+            <box size="0.1 0.1 0.1" />
+         </geometry>
+      </collision>
+      <visual name="hokuyo_visual">
+         <origin xyz="0 0 0" rpy="0 0 0" />
+         <geometry>
+            <mesh filename="package://my_robot/meshes/hokuyo.dae" />
+         </geometry>
+      </visual>
+   </link>
+   <joint type="fixed" name="hokuyo_joint">
+      <origin xyz="0.15 0 0.1" rpy="0 0 0" />
+      <child link="hokuyo" />
+      <parent link="chassis" />
+      <axis xyz="0 1 0" rpy="0 0 0" />
+      <limit effort="10000" velocity="1000" />
+      <dynamics damping="1.0" friction="1.0" />
+   </joint>
+    <gazebo reference="chassis">
+       <material>Gazebo/Blue</material>
+    </gazebo>
+    <gazebo reference="left_wheel">
+      <material>Gazebo/Green</material>
+    </gazebo>
+    <gazebo reference="right_wheel">
+       <material>Gazebo/Green</material>
+    </gazebo>
+    <gazebo reference="camera">
+       <material>Gazebo/Red</material>
+    </gazebo>
 </robot>

Commit message: feat: added simulated kinect to robot

File: catkin_ws/src/my_robot/urdf/my_robot.xacro (robot description, xacro)
@@ -165,4 +165,12 @@
       <dynamics damping="1.0" friction="1.0" />
    </joint>
+   <!-- Simulated Kinect -->
+    <joint name="camera_optical_joint" type="fixed">
+        <origin xyz="0 0 0" rpy="-1.5707 0 -1.5707"/>
+        <parent link="camera_link"/>
+        <child link="camera_link_optical"/>
+    </joint>
+    <link name="camera_link_optical">
+    </link>
     <!-- Gazebo Materials -->
     <gazebo reference="chassis">

Commit message: feat: added simulated kinect RGB-D Camera

File: catkin_ws/src/my_robot/urdf/my_robot.xacro (robot description, xacro)
@@ -137,4 +137,12 @@
       <dynamics damping="1.0" friction="1.0" />
    </joint>
+    <!-- RGB-D Camera -->
+    <joint name="camera_optical_joint" type="fixed">
+        <origin xyz="0 0 0" rpy="-1.5707 0 -1.5707"/>
+        <parent link="camera"/>
+        <child link="camera_link_optical"/>
+    </joint>
+    <link name="camera_link_optical">
+    </link>
    <!-- Lidar -->
    <link name="hokuyo">
@@ -165,12 +173,4 @@
       <dynamics damping="1.0" friction="1.0" />
    </joint>
-   <!-- Simulated Kinect -->
-    <joint name="camera_optical_joint" type="fixed">
-        <origin xyz="0 0 0" rpy="-1.5707 0 -1.5707"/>
-        <parent link="camera_link"/>
-        <child link="camera_link_optical"/>
-    </joint>
-    <link name="camera_link_optical">
-    </link>
     <!-- Gazebo Materials -->
     <gazebo reference="chassis">
